File: IOT Product Development/Smart_Savour/Smart_Savour.kicad_sch (KiCad schematic)
At the start: 30 parts, among them J1 12V DC, J2 5V DC, J3 DWIN interface, J4 Programming Interface, SW1 SW_Push, SW2 SW_Push, U1 LM1117MP-5, U2 LM1117MP-3.3, U3 ESP32-WROOM-32

Commit message: Updated Schematic Version 2
Parts:
- added C11: 0.1uF_0805, Capacitor_SMD:C_0805_2012Metric_Pad1.18x1.45mm_HandSolder, symbol Device:C_Small
- added C12, C13: 10uF, Capacitor_THT:CP_Radial_D6.3mm_P2.50mm, symbol Device:C_Polarized_US
- added F1: Polyfuse, Package_TO_SOT_SMD:SOT-23-6, symbol Device:Polyfuse
- added J5: USB_C_Receptacle_USB2.0_16P, symbol Connector:USB_C_Receptacle_USB2.0_16P
- added J6: ~, symbol Connector:Screw_Terminal_01x02
- added Q1, Q2: BC817, Package_TO_SOT_SMD:SOT-23, symbol Transistor_BJT:BC817
- added R6, R7, R8, R9: 10k_0805, Resistor_SMD:R_0805_2012Metric_Pad1.20x1.40mm_HandSolder, symbol Device:R_US
- added U4: CH340C, Package_SO:SOIC-16_3.9x9.9mm_P1.27mm, symbol Interface_USB:CH340C
- added U5: WE-TVS-82400102, Package_TO_SOT_SMD:SOT-23-6, symbol Power_Protection:WE-TVS-82400102
Connections:
- net +3.3V: now also C11.1, C12.1, U4.16 (VCC), U4.4 (V3)
- net +5V: now also J6.1 (Pin_1)
- net Boot: now also Q2.2 (E)
- net En: now also Q1.3 (C)
- net GNDREF: now also C11.2, C12.2, C13.2, J5.A1 (GND), J5.A12 (GND), J5.B1 (GND), J5.B12 (GND), J5.S1 (SHIELD), R8.1, R9.1, U4.1 (GND), U5.2
- net Rx: now also U4.2 (TXD)
- net Tx: now also U4.3 (RXD)
- new net: J5.A5 (CC1), R8.2
- new net: F1.2, J6.2 (Pin_2)
- new net: Q1.1 (B), R6.1
- new net: J5.A7 (D-), J5.B7 (D-), U5.1
- new net: J5.A6 (D+), J5.B6 (D+), U5.3
- new net: J5.B5 (CC2), R9.2
- new net: Q2.1 (B), R7.1
- new net +5v Bus: C13.1, F1.1, J5.A4 (VBUS), J5.A9 (VBUS), J5.B4 (VBUS), J5.B9 (VBUS), U5.5
- new net DTR: Q2.3 (C), R6.2, U4.13 (~{DTR})
- new net D_N: U4.6 (UD-), U5.6
- new net D_P: U4.5 (UD+), U5.4
- new net RTS: Q1.2 (E), R7.2, U4.14 (~{RTS})
- no-connect marks 28 -> 35
Other:
- note added: "Auto Programming"
- note added: "External Programming Interface"
- note added: "Type C Interface"
- moved on the sheet: C1, C10, C2, C3, C4, C5, C6, C7, C8, C9, D1, D2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
