File: Iot Product Development/Smart_Savour/Smart_Savour.kicad_pcb (KiCad board)
At the start: 2 copper layers, 44 parts, among them J1 12V DC, J2 5V DC, J3 DWIN interface, J4 Programming Interface, J5 USB_C_Receptacle_USB2.0_16P, Q1 BC817, Q2 BC817, SW1 SW_Push, SW2 SW_Push, U1 LM1117MP-5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

Commit message: Folder updated
Parts:
- moved U3 2.97 mm to (73.7, 72.1)
